File: project/ADIS Teensy Arduino Breakout RevC.sch (EAGLE design)
At the start: 25 parts, among them J1 A3-16PA-2SV(71)T, J2 ARDUINO_R3_SHIELDUNO_R3_SHIEL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, J3 TEENSY-3.1SILK, J4 AVR_SPI_PRG_6PTH, J5 M02PTH, J6 M02PTH, J8 VIN, J9 3V3 EXT, U1 ADP2303, U2 SIP32510

Commit message: Updated BOM in brd and sch files
Parts:
- J1: PARTNO (none) -> A3-16PA-2SV(71)
- J10, J7: PARTNO (none) -> 68000-103HLF
- J3: PARTNO (none) -> TEENSY32
- J4: PARTNO (none) -> M20-9720345
- J9: PARTNO (none) -> 20020327-C021B01LF
- L1: PARTNO (none) -> CLF6045T-6R8N-H
- U2: PARTNO (none) -> SIP32510DT-T1-GE3
Changed lines of the file:
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@@
 <layer number="255" name="routoute" color="7" fill="1" visible="yes" active="yes"/>
 </layers>
-<schematic xreflabel="%F%N/%S" xrefpart="/%S">
+<schematic xreflabel="%F%N/%S.%C%R" xrefpart="/%S.%C%R">
 <attributes>
 </attributes>
@@
 <parts>
 <part name="J2" library="Testing" deviceset="ARDUINO_R3_SHIELD" device="UNO_R3_SHIELD_HOLES"/>
-<part name="J4" library="SparkFun-Connectors" deviceset="AVR_SPI_PRG_6" device="PTH"/>
-<part name="J3" library="Testing" deviceset="TEENSY-3.1" device="SILK"/>
+<part name="J4" library="SparkFun-Connectors" deviceset="AVR_SPI_PRG_6" device="PTH">
+<attribute name="PARTNO" value="M20-9720345"/>
+</part>
+<part name="J3" library="Testing" deviceset="TEENSY-3.1" device="SILK">
+<attribute name="PARTNO" value="TEENSY32"/>
+</part>
 <part name="GND1" library="SparkFun-Aesthetics" deviceset="GND" device=""/>
 <part name="GND2" library="SparkFun-Aesthetics" deviceset="GND" device=""/>
@@
 <attribute name="PARTNO" value="TLJA476M010R0600"/>
 </part>
-<part name="J1" library="Analog Devices iSensors" deviceset="A3-16PA-2SV(71)" device="T"/>
+<part name="J1" library="Analog Devices iSensors" deviceset="A3-16PA-2SV(71)" device="T">
+<attribute name="PARTNO" value="A3-16PA-2SV(71)"/>
+</part>
 <part name="GND4" library="SparkFun-Aesthetics" deviceset="GND" device=""/>
-<part name="J7" library="SparkFun-Connectors" deviceset="M03" device="PTH"/>
+<part name="J7" library="SparkFun-Connectors" deviceset="M03" device="PTH">
+<attribute name="PARTNO" value="68000-103HLF"/>
+</part>
 <part name="D2" library="Chong" deviceset="DIODE-" device="DO214AA" value="SSB43L-E3">
 <attribute name="PARTNO" value="SSB43L-E3/52T"/>
 </part>
-<part name="L1" library="AnalogDevices" deviceset="CLF6045T-6R8N-H" device=""/>
+<part name="L1" library="AnalogDevices" deviceset="CLF6045T-6R8N-H" device="">
+<attribute name="PARTNO" value="CLF6045T-6R8N-H"/>
+</part>
 <part name="SUPPLY8" library="SparkFun-Aesthetics" deviceset="5V" device=""/>
 <part name="FRAME1" library="frames_Juan" deviceset="FRAME_A_L" device=""/>
 <part name="FRAME2" library="frames_Juan" deviceset="FRAME_A_L" device=""/>
-<part name="J9" library="SparkFun-Connectors" deviceset="CONN_02" device="3.5MM" value="3V3 EXT"/>
-<part name="U2" library="Chong" deviceset="SIP32510" device=""/>
+<part name="J9" library="SparkFun-Connectors" deviceset="CONN_02" device="3.5MM" value="3V3 EXT">
+<attribute name="PARTNO" value="20020327-C021B01LF"/>
+</part>
+<part name="U2" library="Chong" deviceset="SIP32510" device="">
+<attribute name="PARTNO" value="SIP32510DT-T1-GE3"/>
+</part>
 <part name="GND5" library="SparkFun-Aesthetics" deviceset="GND" device=""/>
 <part name="GND6" library="SparkFun-Aesthetics" deviceset="GND" device=""/>
-<part name="J10" library="SparkFun-Connectors" deviceset="CONN_03" device=""/>
+<part name="J10" library="SparkFun-Connectors" deviceset="CONN_03" device="">
+<attribute name="PARTNO" value="68000-103HLF"/>
+</part>
 <part name="SUPPLY4" library="SparkFun-Aesthetics" deviceset="3.3V" device=""/>
 </parts>
@@
 <instance part="J4" gate="G$1" x="66.04" y="38.1" smashed="yes">
 <attribute name="NAME" x="61.722" y="43.942" size="1.778" layer="95"/>
-</instance>
-<instance part="J3" gate="G$1" x="210.82" y="129.54"/>
+<attribute name="PARTNO" x="66.04" y="38.1" size="1.778" layer="96" display="off"/>
+</instance>
+<instance part="J3" gate="G$1" x="210.82" y="129.54">
+<attribute name="PARTNO" x="210.82" y="129.54" size="1.778" layer="96" display="off"/>
+</instance>
 <instance part="GND1" gate="1" x="78.74" y="78.74"/>
 <instance part="GND2" gate="1" x="182.88" y="93.98"/>
@@
 <attribute name="NAME" x="134.62" y="28.702" size="1.778" layer="95"/>
 </instance>
-<instance part="J1" gate="J$1" x="43.18" y="177.8"/>
+<instance part="J1" gate="J$1" x="43.18" y="177.8">
+<attribute name="PARTNO" x="43.18" y="177.8" size="1.778" layer="96" display="off"/>
+</instance>
 <instance part="GND4" gate="1" x="55.88" y="154.94"/>
 <instance part="FRAME1" gate="G$1" x="0" y="0"/>
 <instance part="FRAME1" gate="G$2" x="172.72" y="0"/>
-<instance part="J9" gate="G$1" x="139.7" y="160.02" rot="R180"/>
-<instance part="U2" gate="U$1" x="96.52" y="172.72"/>
+<instance part="J9" gate="G$1" x="139.7" y="160.02" rot="R180">
+<attribute name="PARTNO" x="139.7" y="160.02" size="1.778" layer="96" display="off"/>
+</instance>
+<instance part="U2" gate="U$1" x="96.52" y="172.72">
+<attribute name="PARTNO" x="96.52" y="172.72" size="1.778" layer="96" display="off"/>
+</instance>
 <instance part="GND5" gate="1" x="109.22" y="165.1"/>
 <instance part="GND6" gate="1" x="129.54" y="152.4"/>
-<instance part="J10" gate="J$1" x="139.7" y="175.26" rot="R180"/>
+<instance part="J10" gate="J$1" x="139.7" y="175.26" rot="R180">
+<attribute name="PARTNO" x="139.7" y="175.26" size="1.778" layer="96" display="off"/>
+</instance>
 <instance part="SUPPLY4" gate="G$1" x="129.54" y="180.34"/>
 </instances>
@@
 <attribute name="PARTNO" x="119.38" y="106.68" size="1.778" layer="96" display="off"/>
 </instance>
-<instance part="J7" gate="G$1" x="88.9" y="129.54"/>
+<instance part="J7" gate="G$1" x="88.9" y="129.54">
+<attribute name="PARTNO" x="88.9" y="129.54" size="1.778" layer="96" display="off"/>
+</instance>
 <instance part="D2" gate="G$1" x="106.68" y="132.08" smashed="yes" rot="R180">
 <attribute name="NAME" x="101.092" y="136.3726" size="1.778" layer="95"/>
@@
 <attribute name="NAME" x="177.8" y="115.57" size="1.778" layer="95"/>
 <attribute name="VALUE" x="177.8" y="113.03" size="1.778" layer="96"/>
+<attribute name="PARTNO" x="180.34" y="111.76" size="1.778" layer="96" display="off"/>
 </instance>
 <instance part="SUPPLY8" gate="G$1" x="119.38" y="134.62"/>
