File: project/ADIS_Teensy_Arduino Breakout RevD.brd (EAGLE design)
At the start: 53.3 x 59.7 mm, 23 parts, among them J1 A3-16PA-2SV(71)T, J2 ARDUINO_R3_SHIELDUNO_R3_SHIEL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, J3 TEENSY-3.1SILK, J4 AVR_SPI_PRG_6PTH, J5 M02PTH, J6 M02PTH, J8 VIN, J9 POWER_JACKPTH_LOCK, U1 ADP2303

Commit message: Updated PCB to Rev D
Parts:
- added J10: (no value), SparkFun-Connectors:1X03
- added J11: M02PTH, SparkFun-Connectors:1X02@1
- added U2: SIP32510, Chong:SOT23-6
- J5, J6: device SparkFun-Connectors:1X02 -> SparkFun-Connectors:1X02@1
- J7: device SparkFun-Connectors:1X03 -> SparkFun-Connectors:1X03@1
- J8: device SparkFun-Connectors:SCREWTERMINAL-3.5MM-2 -> SparkFun-Connectors:SCREWTERMINAL-3.5MM-2@1
- J9: value POWER_JACKPTH_LOCK -> 3V3 EXT; device SparkFun-Connectors:POWER_JACK_PTH_LOCK -> SparkFun-Connectors:SCREWTERMINAL-3.5MM-2
- moved J9 59.4 mm to (38.9, 72.1)
- moved J8 8.44 mm to (47.0, 22.4)
- moved SJ1 6.86 mm to (46.4, 62.7)
- moved SJ2 6.86 mm to (46.4, 60.4)
- moved J7 1.70 mm to (52.6, 30.0)
Connections:
- new net N$10: J10.3, J9.1
- new net N$11: J10.2, J11.2, U2.5, U2.6
- new net N$8: J1.10, J1.11, J1.12, J11.1, U2.1, U2.2
- net 3.3V: now also J10.1; no longer J1.10, J1.11, J1.12
- net D7: now also U2.3
- net GND: now also J9.2, U2.4; no longer J9.GND, J9.GNDBREAK
- net VIN: no longer J9.PWR
Routing:
- net D7: track 46.3 -> 94.9 mm
- net N$8: track 0.00 -> 37.4 mm, vias 0 -> 2
- net N$11: track 0.00 -> 34.9 mm
- net 3.3V: track 64.0 -> 82.4 mm, vias 4 -> 5
- net VIN: track 46.9 -> 37.6 mm
- net N$10: track 0.00 -> 6.73 mm
- net A5: track 9.00 -> 15.6 mm
- net SDA: track 80.1 -> 74.7 mm
- net A6: track 67.2 -> 61.8 mm
- net SCL: track 79.5 -> 74.5 mm
- net A7: track 61.1 -> 56.8 mm
- net A4: track 14.8 -> 12.0 mm, vias 0 -> 1
- net RESET: track 58.3 -> 55.8 mm
- net D2: track 98.3 -> 100.4 mm
- net A2: track 47.5 -> 49.1 mm
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Other:
- board text added: "3.3V"
- board text added: "Juan Chong"
- board text added: "ONLY!"
- board text added: "REG"
- board text added: "RevD-02/2019"
- board text added: "SWBP"
- board text removed: "JChong"
- board text removed: "RevB-10/2016"
- board text removed: "VIN"
