File: project/ADIS_Teensy_Arduino Breakout RevD.sch (EAGLE design)
At the start: 23 parts, among them J1 A3-16PA-2SV(71)T, J2 ARDUINO_R3_SHIELDUNO_R3_SHIEL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, J3 TEENSY-3.1SILK, J4 AVR_SPI_PRG_6PTH, J5 M02PTH, J6 M02PTH, J8 VIN, J9 POWER_JACKPTH_LOCK, U1 ADP2303

Commit message: Updated PCB to Rev D
Parts:
- added J10: (no value), SparkFun-Connectors:CONN_03
- added J11: M02PTH, SparkFun-Connectors:M02PTH
- added U2: SIP32510, Chong:SIP32510
- J1: PARTNO (none) -> A3-16PA-2SV(71)
- J3: PARTNO (none) -> TEENSY32
- J4: PARTNO (none) -> M20-9720345
- J7: PARTNO (none) -> 68000-103HLF
- J9: value POWER_JACKPTH_LOCK -> 3V3 EXT; device SparkFun-Connectors:POWER_JACKPTH_LOCK -> SparkFun-Connectors:CONN_023.5MM; PARTNO (none) -> 20020327-C021B01LF
- L1: PARTNO (none) -> CLF6045T-6R8N-H
Connections:
- new net N$10: J10.3, J9.1
- new net N$11: J10.2, J11.2, U2.IN@1, U2.IN@2
- new net N$8: J1.VDD@1, J1.VDD@2, J1.VDD@3, J11.1, U2.OUT@1, U2.OUT@2
- net 3.3V: now also J10.1; no longer J1.VDD@1, J1.VDD@2, J1.VDD@3
- net D7: now also U2.EN
- net GND: now also J9.2, U2.GND; no longer J9.GND, J9.GNDBREAK
- net VIN: no longer J9.PWR
Other:
- note added: "Analog Switch Bypass"
- moved on the sheet: J1
